Commit message: Changes made to ball_chaser->process_image.cpp, my_robot->my_robot.xacro, my_robot->Office.world

File: .Project2/my_robot/urdf/my_robot.xacro (robot description, xacro)
@@ -179,14 +179,14 @@
   <!-- COLOR DEFINITIONS -->
   <gazebo reference="camera">
-    <material>Gazebo/Red</material>
+    <material>Gazebo/Blue</material>
   </gazebo>
   <gazebo reference="left_wheel">
-    <material>Gazebo/Green</material>
+    <material>Gazebo/Purple</material>
   </gazebo>
   <gazebo reference="right_wheel">
-    <material>Gazebo/Green</material>
+    <material>Gazebo/Purple</material>
   </gazebo>
   <gazebo reference="chassis">
-    <material>Gazebo/Blue</material>
+    <material>Gazebo/Yellow</material>
   </gazebo>
 </robot>
